Commit message: changed position of camera to be held in gripper

File: software/ros_packages/rover_arm/config/rover_arm.urdf.xacro (robot description, xacro)
@@ -12,5 +12,5 @@
     <!-- Instantiate micros  -->
     <xacro:sensor_d405 parent ="arm_gripper" name="camera" use_nominal_extrinsics="true">
-        <origin xyz="0 0.05 0.1" rpy="-1.5707 -1.5707 0"/>
+        <origin xyz="0.0175 0.0 0.2" rpy= "0 -1.5707 0"/>
     </xacro:sensor_d405>
     <xacro:rover_arm_ros2_control name="RealSystem" initial_positions_file="$(arg initial_positions_file)" ros2_control_hardware_type="$(arg ros2_control_hardware_type)"/>

Commit message: Added controller switching

File: software/ros_packages/rover_arm/config/rover_arm.urdf.xacro (robot description, xacro)
@@ -12,5 +12,5 @@
     <!-- Instantiate micros  -->
     <xacro:sensor_d405 parent ="arm_gripper" name="camera" use_nominal_extrinsics="true">
-        <origin xyz="0.0175 0.0 0.2" rpy= "0 -1.5707 0"/>
+        <origin xyz="0 0.05 0.1" rpy="-1.5707 -1.5707 0"/>
     </xacro:sensor_d405>
     <xacro:rover_arm_ros2_control name="RealSystem" initial_positions_file="$(arg initial_positions_file)" ros2_control_hardware_type="$(arg ros2_control_hardware_type)"/>
